File: XT302+2 PCB mod/XT302+2 PCB mod.kicad_pcb (KiCad board)
At the start: 2 copper layers, 20.4 x 25 mm, 27 parts

Commit message: Hotfix to v2
Parts:
- removed the 2plus2: Hirose_DF13-02P-1.25DSA_1x02_P1.25mm_Vertical, Connector_Hirose:Hirose_DF13-02P-1.25DSA_1x02_P1.25mm_Vertical (x3)
- added REF**: PinHeader_1x02_P2.00mm_Vertical, Connector_PinHeader_2.00mm:PinHeader_1x02_P2.00mm_Vertical, F.Cu at (196.0, 149.0)
- added REF**: PinHeader_1x02_P2.00mm_Vertical, Connector_PinHeader_2.00mm:PinHeader_1x02_P2.00mm_Vertical, F.Cu at (195.9, 141.5)
- added REF**: PinHeader_1x02_P2.00mm_Vertical, Connector_PinHeader_2.00mm:PinHeader_1x02_P2.00mm_Vertical, F.Cu at (195.9, 133.5)
